File: PCB_Related/MaxAir_Smart_Home_Gateway_WT21-ET01-v095/MaxAir_Smart_Home_Gateway_WT21-ET01-v095.sch (EAGLE design)
At the start: 27 parts, among them J2 DCJ0202

Commit message: MaxAir Smart Home Gateway
MaxAir Smart Home Gateway updates:
micro usb smd connector added, and power line traces width increased.
Parts:
- added IC2: HT7333, holtek2:HT7333
- added SJ1: (no value), jumper:SJ
- added U$3: MICRO-USB, microusb:MICRO-USB
Connections:
- new net VCC_RADIO: C1.+, C2.1, IC2.OUT, JP1.2, JP2.2, SJ1.1
- net GND: now also IC2.GND, U$3.GND, U$3.GND@1, U$3.GND@2
- net VCC_3.3: now also SJ1.2; no longer C1.+, C2.1, JP1.2, JP2.2
- net VCC_5: now also IC2.IN, U$3.VCC
Other:
- note added: "Last Update: 22/07/2022 00:58"
- note removed: "Last Update: 167/03/2022 00:28"
- moved on the sheet: C1, C2, C3, C4
